File: Meno/Schematic/Meno_01.sch (KiCad schematic (older format))
At the start: 21 parts, among them J2 AVR-ISP-6, J4 Conn_02x19_Female, J5 Conn_02x12_Female, J6 Conn_02x15_Female, SW1 B3FS-1050P, U1 ATmega2560-16AUR, Y1 FA238-16MHz

Commit message: ピンソケットの構成を変更
Parts:
- removed J4: Conn_02x19_Female, Connector_PinSocket_2.54mm:PinSocket_2x19_P2.54mm_Vertical, symbol Connector_Generic:Conn_02x19_Odd_Even
- removed J6: Conn_02x15_Female, Connector_PinSocket_2.54mm:PinSocket_2x15_P2.54mm_Vertical, symbol Connector_Generic:Conn_02x15_Odd_Even
- added J4, J8: Conn_01x08, Connector_PinSocket_2.54mm:PinSocket_1x08_P2.54mm_Vertical, symbol Connector_Generic:Conn_01x08
- added J5: Conn_01x10, Connector_PinSocket_2.54mm:PinSocket_1x10_P2.54mm_Vertical, symbol Connector_Generic:Conn_01x10
- added J6: Conn_01x19, Connector_PinSocket_2.54mm:PinSocket_1x19_P2.54mm_Vertical, symbol Connector_Generic:Conn_01x19
- added J7: Conn_01x06, Connector_PinSocket_2.54mm:PinSocket_1x06_P2.54mm_Vertical, symbol Connector_Generic:Conn_01x06
- added J9: Conn_01x15, Connector_PinSocket_2.54mm:PinSocket_1x15_P2.54mm_Vertical, symbol Connector_Generic:Conn_01x15
- C1, C2, C3, C4, C5, C6, C7: footprint Capacitor_SMD:C_0805_2012Metric -> Capacitor_SMD:C_0805_2012Metric_Pad1.15x1.40mm_HandSolder
- D1: footprint LED_SMD:LED_0805_2012Metric -> LED_SMD:LED_0805_2012Metric_Pad1.15x1.40mm_HandSolder
- D5: footprint Diode_SMD:D_SOD-123 -> SOD123(F)-HandSolder:D_SOD-123
- J10: renamed from J5; value Conn_02x12_Female -> Conn_02x12
- L1: footprint Inductor_SMD:L_0805_2012Metric -> Inductor_SMD:L_0805_2012Metric_Pad1.15x1.40mm_HandSolder
- R1, R2, R3, R4: footprint Resistor_SMD:R_0805_2012Metric -> Resistor_SMD:R_0805_2012Metric_Pad1.15x1.40mm_HandSolder
Connections:
- no-connect marks 20 -> 18
Other:
- moved on the sheet: J10
