File: Meno/PCB_Layout/Meno.kicad_pcb (KiCad board)
At the start: 2 copper layers, 68.5 x 53.3 mm, 49 parts, among them J1 5077CR-16SMC2, J2 AVR-ISP-6, J3 18742, J4 Conn_02x19_Female, J5 Conn_02x12_Female, J6 Conn_02x15_Female, Q1 IRLML6402, SW1 B3FS-1050P, U1 ATmega2560-16AUR, U2 FT232RL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

Commit message: 0ecd643での変更を基板データに反映
Parts:
- added J10: Conn_02x12, Connector_PinSocket_2.54mm:PinSocket_2x12_P2.54mm_Vertical, F.Cu at (170.9, 88.3)
- added J7: Conn_01x06, Connector_PinSocket_2.54mm:PinSocket_1x06_P2.54mm_Vertical, F.Cu at (177.7, 125.8)
- added J8: Conn_01x08, Connector_PinSocket_2.54mm:PinSocket_1x08_P2.54mm_Vertical, F.Cu at (159.9, 125.8)
- added J9: Conn_01x15, Connector_PinSocket_2.54mm:PinSocket_1x15_P2.54mm_Vertical, F.Cu at (177.7, 123.3)
- added MH1: Mount_TH_3.2mm_NoWasher, Mount_TH_3.2mm_NoWasher:Mount_TH_3.2mm_NoWasher, F.Cu at (185.8, 92.8)
- added MH2: Mount_TH_3.2mm_NoWasher, Mount_TH_3.2mm_NoWasher:Mount_TH_3.2mm_NoWasher, F.Cu at (185.8, 120.7)
- added MH3: Mount_TH_3.2mm_NoWasher, Mount_TH_3.2mm_NoWasher:Mount_TH_3.2mm_NoWasher, F.Cu at (129.3, 70.8)
- added MH4: Mount_TH_3.2mm_NoWasher, Mount_TH_3.2mm_NoWasher:Mount_TH_3.2mm_NoWasher, F.Cu at (128.3, 131.8)
- J4: value Conn_02x19_Female -> Conn_01x08; footprint Connector_PinSocket_2.54mm:PinSocket_2x19_P2.54mm_Vertical -> Connector_PinSocket_2.54mm:PinSocket_1x08_P2.54mm_Vertical
- J5: value Conn_02x12_Female -> Conn_01x10; footprint Connector_PinSocket_2.54mm:PinSocket_2x12_P2.54mm_Vertical -> Connector_PinSocket_2.54mm:PinSocket_1x10_P2.54mm_Vertical
- J6: value Conn_02x15_Female -> Conn_01x19; footprint Connector_PinSocket_2.54mm:PinSocket_2x15_P2.54mm_Vertical -> Connector_PinSocket_2.54mm:PinSocket_1x19_P2.54mm_Vertical
- ZLS1: renamed from G***; value LOGO -> Amateur Intent Logo (Designed by @MakoTr_01)
- moved J6 45.7 mm to (177.7, 80.1)
- moved J5 18.4 mm to (155.9, 77.6), turned to 270 degrees
- moved C6 8.27 mm to (147.2, 89.0), turned to 270 degrees
- moved C7 8.27 mm to (155.5, 89.0), turned to 90 degrees
- moved J4 2.54 mm to (177.7, 77.6)
- moved C12 0.67 mm to (132.3, 123.5)
- moved C13 0.66 mm to (138.5, 123.6)
- renumbered C7 to C6, C6 to C7, REF** to ZLS2
Connections:
- C6 pad 2: Net-(C7-Pad2) -> Net-(C6-Pad2)
- C7 pad 2: Net-(C6-Pad2) -> Net-(C7-Pad2)
- J4 pad 1: D32 -> D0
- J4 pad 2: D0 -> D1
- J4 pad 3: D31 -> D2
- J4 pad 4: D1 -> D3
- J4 pad 5: D30 -> D4
- J4 pad 6: D2 -> D5
- J4 pad 7: D29 -> D6
- J4 pad 8: D3 -> D7
- J5 pad 1: D43 -> D8
- J5 pad 10: D50 -> D21
- J5 pad 2: VCC -> D9
- J5 pad 3: D42 -> D10
- J5 pad 4: D53 -> D11
- J5 pad 5: D41 -> D12
- J5 pad 6: D52 -> D13
- J5 pad 7: D40 -> GND
- J5 pad 8: D51 -> AREF
- J5 pad 9: D39 -> D20
- J6 pad 1: A5 -> D32
- J6 pad 10: A10 -> D23
- J6 pad 11: A0 -> D22
- J6 pad 12: A11 -> D21
- J6 pad 13: Net-(J6-Pad13) -> D20
- J6 pad 14: A12 -> D19
- J6 pad 15: VS -> D18
- J6 pad 16: VS -> D17
- J6 pad 17: GND -> D16
- J6 pad 18: GND -> D15
- J6 pad 19: GND -> D14
- J6 pad 2: A6 -> D31
- J6 pad 3: A4 -> D30
- J6 pad 4: A7 -> D29
- J6 pad 5: A3 -> D28
- J6 pad 6: A8 -> D27
- J6 pad 7: A2 -> D26
- J6 pad 8: A9 -> D25
- J6 pad 9: A1 -> D24
Routing:
- net A5: track 48.4 -> 54.1 mm
- net D21: track 56.2 -> 55.0 mm
- net D12: track 30.4 -> 31.4 mm
- net AREF: track 63.8 -> 64.6 mm
- net GND: vias 14 -> 13
Other:
- outline, holes or cut-outs redrawn
- board text added: "4-Φ3.2"
- board text removed: "Φ3.2 (4x)"
