File: Meno_V101/Schematic/Meno_V101_02.sch (KiCad schematic (older format))
At the start: 24 parts, among them J1 5077CR-16SMC2, J3 18742, Q1 IRLML6402, U2 FT232RQ, U3 LM340MPX-5.0/NOPB, U4 TLV75733PDBVR

Commit message: プリント基板のパターンとシルク位置の変更
Parts:
- C10: value 0.22u -> 0.33u
Changed lines of the file:
@@
 AR Path="/5E4DD525/5F8EB731" Ref="C10"  Part="1"
 F 0 "C10" H 8050 3900 50  0000 L CNN
-F 1 "0.22u" H 8050 3800 50  0000 L CNN
+F 1 "0.33u" H 8050 3800 50  0000 L CNN
 F 2 "Capacitor_SMD:C_0603_1608Metric" H 7988 3700 50  0001 C CNN
 F 3 "https://psearch.jp.murata.com/capacitor/product/GCM21BR71H224KA37%23.html" H 7950 3850 50  0001 C CNN
